File: schematics/Audio.kicad_sch (KiCad schematic)
At the start: 54 parts, among them J1 HEADPHONES, U1 6116, U4 NEO-DO, U7 YM3016D, U8 NJM2066D, X3 24MHz

Commit message: Audio Amp + player's button LED & marquee + Coins Up + 45% raiser card connectors
Parts:
- removed VR (x2): 1K, symbol Device:R_Potentiometer_Small
- added RV1, RV2: 1K, symbol Device:R_Potentiometer_Dual_Separate
- C10, C11, C13, C14, C15, C16, C22, C26, C30, C32, C9: symbol Device:C -> Device:C_Small
- R28, R29, R30, R31, R32, R33, R34, R35, R36, R37, R38, R39, R40: symbol Device:R -> Device:R_Small
Connections:
- net SOMWR is gone; now on net SDMWR: U1.21 (WE)
- net 24M: now also R28.1
- net GND: now also R28.2, RV1.3, RV2.3; no longer C22.2, C26.2, C30.2, C32.2, R36.2
- net at C25.2: now also RV2.2
- net at R29.2: now also C9.1, X3.2
- net at C25.1, U8.1 (INPUT2): no longer C26.1
- net at R37.1: no longer C23.2
- net at R39.2: no longer U8.10 (OUT1)
- net at 2L.27 (ANALOG), C18.1, C20.1: no longer R36.1
- net at C21.2: now also RV1.2
- net at R40.2: no longer U8.7 (OUT2)
- net at C21.1, U8.16 (INPUT1): no longer C22.1
- net at R38.1: no longer C24.2
- net SOMRO renamed SDMRO
- net SORO renamed SDRO
- net SOWR renamed SDWR
- now unconnected: C30.1, C31.1, C32.1, C33.1, R39.1, R40.1
Other:
- title: (none) -> Audio - Z80 NEO-D0
