File: schematics/DaughterBoard.kicad_sch (KiCad schematic)
At the start: 4 parts, among them CN1 DIN41612_03x32_AC, CN7 DIN41612_03x32_AC

Commit message: typos
Parts:
- 1E, 1F: footprint (none) -> Package_DIP:DIP-14_W7.62mm
Other:
- company: (none) -> SNK
Changed lines of the file:
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@@
 (kicad_sch (version 20230121) (generator eeschema)
   (paper "User" 670.814 629.361)
+  (title_block
+    (date "2023-08-15")
+    (company "SNK")
+    (comment 3 "Converted by Frater ")
+    (comment 4 "NEO-GEO MVS MV1F")
+    (comment 9 "https://github.com/Neo-Geo-Hardwares/Schematics-MV1F")
+  )
   (junction (at 127 254) (diameter 0) (color 0 0 0 0)
   )
@@
       (effects (font (size 1.27 1.27)))
     )
-    (property "Footprint" "" (at 52.07 222.25 0)
+    (property "Footprint" "Package_DIP:DIP-14_W7.62mm" (at 52.07 222.25 0)
       (effects (font (size 1.27 1.27)) hide)
     )
@@
       (effects (font (size 1.27 1.27)))
     )
-    (property "Footprint" "" (at 204.47 166.37 0)
+    (property "Footprint" "Package_DIP:DIP-14_W7.62mm" (at 204.47 166.37 0)
       (effects (font (size 1.27 1.27)) hide)
     )
@@
       (effects (font (size 1.27 1.27)))
     )
-    (property "Footprint" "" (at 189.23 163.83 0)
+    (property "Footprint" "Package_DIP:DIP-14_W7.62mm" (at 189.23 163.83 0)
       (effects (font (size 1.27 1.27)) hide)
     )
