File: schematics/lspc2-Vram.kicad_sch (KiCad schematic)
At the start: 15 parts, among them J2 NO

Commit message: Complete Page 2 (LSPC2-A2)
Complete "Main" page LSPC2, NEO-IO, NEO-B1, NEO-ZMC2 & SFix Rom LO Rom
Parts:
- added 1F: NEO-ZMC2, symbol 0-Custom-SNK:NEO-ZMC2
- added 1G: 74LS32, symbol 74xx:74LS32
- added 2D: NEO-IO, symbol 0-Custom-SNK:NEO-IO
- added 2E: 37C301, symbol 0-Custom-SNK:37C301
- added J10, J6: NO, symbol Jumper:SolderJumper_2_Open
- added J5, J9: ~, symbol Jumper:SolderJumper_2_Bridged
- added JAMMAF: SYNC, symbol Connector:Conn_01x01_Pin
- added R26: 100, symbol Device:R_Small_US
- added R27: 470, symbol Device:R_Small_US
Connections:
- net 2H1: now also 2E.9 (A3)
- net A1: now also 2D.61 (A1)
- net A2: now also 2D.62 (A2)
- net A3: now also 2D.63 (A3)
- net A7: now also 2D.60 (A7)
- net CA4: now also 1F.17 (C4)
- net DOTA: now also 1F.4 (DOTA)
- net DOTB: now also 1F.9 (DOTB)
- net EVEN1: now also J10.1 (A)
- net EVEN2: now also J9.1 (A)
- net FIXD0: now also 2E.13 (D0)
- net FIXD1: now also 2E.14 (D1)
- net FIXD2: now also 2E.15 (D2)
- net FIXD3: now also 2E.17 (D3)
- net FIXD4: now also 2E.18 (D4)
- net FIXD5: now also 2E.19 (D5)
- net FIXD6: now also 2E.20 (D6)
- net FIXD7: now also 2E.21 (D7)
- net GAD0: now also 1F.79 (GAD0)
- net GAD1: now also 1F.80 (GAD1)
- net GAD2: now also 1F.1 (GAD2)
- net GAD3: now also 1F.3 (GAD3)
- net GAD4: now also 1F.10 (GBD0)
- net GAD5: now also 1F.11 (GDB1)
- net GAD6: now also 1F.13 (GDB2)
- net GAD7: now also 1F.14 (GDB3)
- net GND: now also 1F.12 (GND), 1F.2 (GND), 1F.23 (GND), 1F.42 (GND), 1F.52 (GND), 1F.63 (GND), 1F.65 (SDA8), 1F.66 (SDA9), 1F.67 (SDA10), 1F.68 (SDA11), 1F.69 (SDA12), 1F.70 (SDA13), 1F.71 (SDA14), 1F.72 (SDA15), 1F.74 (SDA0), 1F.75 (SDA1), 1F.76 (SDRD0), 1F.77 (CS), 1F.78 (CSDOT), 2D.10 (GND), 2D.23 (SYNCREV), 2D.25 (GND), 2D.34 (SLOT0), 2D.35 (SLOT1), 2D.42 (GND), 2D.57 (GND), 2E.24 (OE)
- net H: now also 1F.7 (H)
- net LOAD: now also 1F.5 (LOAD)
- net P0: now also 2D.2 (P0)
- net P1: now also 2D.3 (P1)
- net P10: now also 2D.38 (P10)
- net P11: now also 2D.48 (P11)
- net P12: now also 2D.49 (P12)
- net P13: now also 2D.50 (P13)
- net P14: now also 2D.51 (P14)
- net P15: now also 2D.52 (P15)
- net P2: now also 2D.4 (P2)
- net P3: now also 2D.5 (P3)
- net P4: now also 2D.15 (P4)
- net P5: now also 2D.16 (P5)
- net P6: now also 2D.17 (P6)
- net P7: now also 2D.18 (P7)
- net P8: now also 2D.36 (P8)
- net P9: now also 2D.37 (P9)
- net PCK2B: now also 2D.1 (PCK2B)
- net RESET: now also 2D.59 (RESET)
- net R/W: now also 2D.32 (RW)
- net SYNC: now also 2D.22 (SYNCIN)
- net VCC: now also 1F.33 (VCC), 1F.73 (VCC), 2D.26 (VCC), 2D.58 (VCC), 2E.1 (VPP), 2E.30 (NC), 2E.31 (PGM), R27.1
- new net: JAMMAF.F (Pin_F), R26.2, R27.2
- new net: 1G.4, 1G.5, J10.2 (B), J5.1 (A), J9.2 (B)
- new net: 1G.6, J6.1 (A)
- new net: 1F.6 (EVEN), J5.2 (B), J6.2 (B)
- new net: 2D.11 (Q05), 2E.26 (A9)
- new net: 2D.12 (Q06), 2E.23 (A10)
- new net: 2D.13 (Q07), 2E.25 (A11)
- new net: 2D.14 (Q08), 2E.4 (A12)
- new net: 2D.24 (SYNCOUT), R26.1
- new net: 2D.39 (Q11), 2E.28 (A13)
- new net: 2D.40 (Q12), 2E.29 (A14)
- new net: 2D.41 (Q13), 2E.3 (A15)
- new net: 2D.43 (Q14), 2E.2 (A16)
- new net: 2D.44 (Q15), 2E.12 (A0)
- new net: 2D.45 (Q16), 2E.11 (A1)
- new net: 2D.46 (Q17), 2E.10 (A2)
- new net: 2D.47 (Q48), 2E.8 (A4)
- new net: 2D.6 (Q01), 2E.7 (A5)
- new net: 2D.7 (Q02), 2E.6 (A6)
- new net: 2D.8 (Q03), 2E.5 (A7)
- new net: 2D.9 (Q04), 2E.27 (A8)
- new net 12M: 1F.50 (12M)
- new net CA0: 1F.15 (C0)
- new net CA1: 1F.19 (C1)
- new net CA10: 1F.25 (C10)
- new net CA11: 1F.29 (C11)
- new net CA12: 1F.26 (C12)
- new net CA13: 1F.30 (C13)
- new net CA14: 1F.27 (C14)
- new net CA15: 1F.31 (C15)
- new net CA16: 1F.32 (C16)
- new net CA17: 1F.37 (C17)
- new net CA18: 1F.34 (C18)
- new net CA19: 1F.38 (C19)
- new net CA2: 1F.16 (C2)
- new net CA20: 1F.35 (C20)
- new net CA21: 1F.39 (C21)
- new net CA22: 1F.36 (C22)
- new net CA23: 1F.40 (C23)
- new net CA24: 1F.41 (C24)
- new net CA25: 1F.46 (C25)
- new net CA26: 1F.43 (C26)
- new net CA27: 1F.47 (C27)
- new net CA28: 1F.44 (C28)
- new net CA29: 1F.48 (C29)
- new net CA3: 1F.20 (C3)
- new net CA30: 1F.45 (C30)
- new net CA31: 1F.49 (C31)
- new net CA5: 1F.21 (C5)
- new net CA6: 1F.18 (C6)
- new net CA7: 1F.22 (C7)
- new net CA8: 1F.24 (C8)
- new net CA9: 1F.28 (C9)
- new net COUNTOUT: 2D.64 (COUNTOUT)
- new net LOCK1: 2D.55 (Q23)
- new net LOCK2: 2D.56 (Q24)
- new net METER1: 2D.53 (Q21)
- new net METER2: 2D.54 (Q22)
- new net PORTADRS: 2D.33 (PORTADRS)
- new net ROMOE: 2D.29 (ROMOE)
- new net ROMOEL: 2D.31 (ROMOEL)
- new net ROMOEU: 2D.30 (ROMOEU)
- new net ROMOH: 2D.20 (ORI1)
- new net SM1CS: 2D.21 (ORO1)
- new net SYSTEH: 2D.19 (ORI0), 2E.22 (CS)
Other:
- moved on the sheet: 1B, 2B, 3E, 4B1, 4C, 5B1, 5ED, 5EE, 5EF, 6C, 6D, J2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

Commit message: Complete pages 1-4
completion of pages 1 to 4
Parts:
- added C221 (x3), C331: 220pF, symbol Device:C
- added C6, C7, C8: 100pF, symbol Device:C
- PAL, R1863, R26, R27, R5814: symbol Device:R_Small_US -> Device:R
Connections:
- net GND: now also C221.2, C221.2, C221.2, C331.2, C6.2, C7.2, C8.2
- net VCC: no longer 2E.30 (NC)
- net 8MB renamed 6MB
- new net LSPC2-A2 146 pin (RESETP): C8.1
- new net NEO-B1 84 pin (1MB): C221.1
- new net NEO-B1 85 pin (CHBL): C221.1
- new net NEO-B1 86 pin (1H1): C221.1
- new net NEO-B1 92 pin (BNKB): C331.1
- new net NEO-B1 96 pin (PCK1): C6.1
- new net NEO-B1 97 pin (PCK2): C7.1
Other:
- company: (none) -> SNK

Commit message: Audio Amp + player's button LED & marquee + Coins Up + 45% raiser card connectors
Parts:
- C221, C331, C6, C7, C8: symbol Device:C -> Device:C_Small
- PAL, R1863, R26, R27, R5814: symbol Device:R -> Device:R_Small
Connections:
- net VCC: no longer R27.1
- net at 2D.24 (SYNCOUT): no longer R26.1
- net SYSTEH renamed SYSTEM
- now unconnected: JAMMAF.F (Pin_F), R26.2, R27.2
Other:
- title: (none) -> LSPC2-A2

Commit message: typos
Parts:
- 1B: footprint (none) -> Package_DIP:DIP-20_W7.62mm
- 1G, 5E: footprint (none) -> Package_DIP:DIP-14_W7.62mm
Changed lines of the file:
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@@
     (comment 3 "Converted by Frater ")
     (comment 4 "NEO-GEO MVS MV1F")
+    (comment 9 "https://github.com/Neo-Geo-Hardwares/Schematics-MV1F")
   )
   (junction (at 445.77 128.27) (diameter 0) (color 0 0 0 0)
@@
       (effects (font (size 1.27 1.27)))
     )
-    (property "Footprint" "" (at 252.73 133.35 0)
+    (property "Footprint" "Package_DIP:DIP-14_W7.62mm" (at 252.73 133.35 0)
       (effects (font (size 1.27 1.27)) hide)
     )
@@
       (effects (font (size 1.27 1.27)))
     )
-    (property "Footprint" "" (at 325.12 148.59 0)
+    (property "Footprint" "Package_DIP:DIP-14_W7.62mm" (at 325.12 148.59 0)
       (effects (font (size 1.27 1.27)) hide)
     )
@@
       (effects (font (size 1.27 1.27)) (justify right))
     )
-    (property "Footprint" "" (at 262.89 68.58 0)
+    (property "Footprint" "Package_DIP:DIP-20_W7.62mm" (at 262.89 68.58 0)
       (effects (font (size 1.27 1.27)) hide)
     )
@@
       (effects (font (size 1.27 1.27)))
     )
-    (property "Footprint" "" (at 252.73 148.59 0)
+    (property "Footprint" "Package_DIP:DIP-14_W7.62mm" (at 252.73 148.59 0)
       (effects (font (size 1.27 1.27)) hide)
     )
@@
       (effects (font (size 1.27 1.27)))
     )
-    (property "Footprint" "" (at 252.73 163.83 0)
+    (property "Footprint" "Package_DIP:DIP-14_W7.62mm" (at 252.73 163.83 0)
       (effects (font (size 1.27 1.27)) hide)
     )
