File: schematics/MV1F-MB-clock.kicad_sch (KiCad schematic)
At the start: 5 parts, among them U3 UPD4990AC, X1 32.768KHz

Commit message: complete DaughterBoard
rename sub files
Parts:
- renumbered C2 to C?, C3 to C?, U3 to U?, X1 to X?
Changed lines of the file:
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@@
   (symbol (lib_id "power:GND") (at 45.72 64.77 0) (unit 1)
     (in_bom yes) (on_board yes) (dnp no) (fields_autoplaced)
-    (property "Reference" "#PWR025" (at 45.72 71.12 0)
+    (property "Reference" "#PWR?" (at 45.72 71.12 0)
       (effects (font (size 1.27 1.27)) hide)
     )
@@
       (project "MVS"
         (path "/8d0803ab-15ed-47a7-8dcb-ab27dc5b29c2"
-          (reference "#PWR025") (unit 1)
+          (reference "#PWR?") (unit 1)
         )
         (path "/8d0803ab-15ed-47a7-8dcb-ab27dc5b29c2/225eaee9-8f74-4a38-a94f-717f461ecd54"
@@
   (symbol (lib_id "Device:C_Small") (at 104.14 46.99 90) (unit 1)
     (in_bom yes) (on_board yes) (dnp no) (fields_autoplaced)
-    (property "Reference" "C2" (at 104.1463 41.2836 90)
+    (property "Reference" "C?" (at 104.1463 41.2836 90)
       (effects (font (size 1.27 1.27)) hide)
     )
@@
       (project "MVS"
         (path "/8d0803ab-15ed-47a7-8dcb-ab27dc5b29c2"
-          (reference "C2") (unit 1)
+          (reference "C?") (unit 1)
         )
         (path "/8d0803ab-15ed-47a7-8dcb-ab27dc5b29c2/225eaee9-8f74-4a38-a94f-717f461ecd54"
@@
   (symbol (lib_id "0-Custom-SNK:UPD4990AC") (at 64.77 46.99 0) (unit 1)
     (in_bom yes) (on_board yes) (dnp no)
-    (property "Reference" "U3" (at 59.69 33.02 0)
+    (property "Reference" "U?" (at 59.69 33.02 0)
       (effects (font (size 1.27 1.27)))
     )
@@
       (project "MVS"
         (path "/8d0803ab-15ed-47a7-8dcb-ab27dc5b29c2"
-          (reference "U3") (unit 1)
+          (reference "U?") (unit 1)
         )
         (path "/8d0803ab-15ed-47a7-8dcb-ab27dc5b29c2/225eaee9-8f74-4a38-a94f-717f461ecd54"
@@
   (symbol (lib_id "Device:Crystal") (at 86.36 52.07 90) (unit 1)
     (in_bom yes) (on_board yes) (dnp no) (fields_autoplaced)
-    (property "Reference" "X1" (at 89.6874 50.8579 90)
+    (property "Reference" "X?" (at 89.6874 50.8579 90)
       (effects (font (size 1.27 1.27)) (justify right))
     )
@@
       (project "MVS"
         (path "/8d0803ab-15ed-47a7-8dcb-ab27dc5b29c2"
-          (reference "X1") (unit 1)
+          (reference "X?") (unit 1)
         )
         (path "/8d0803ab-15ed-47a7-8dcb-ab27dc5b29c2/225eaee9-8f74-4a38-a94f-717f461ecd54"
@@
   (symbol (lib_id "Device:C_Trim_Small") (at 104.14 57.15 90) (unit 1)
     (in_bom yes) (on_board yes) (dnp no) (fields_autoplaced)
-    (property "Reference" "C3" (at 104.013 51.4563 90)
+    (property "Reference" "C?" (at 104.013 51.4563 90)
       (effects (font (size 1.27 1.27)) hide)
     )
@@
       (project "MVS"
         (path "/8d0803ab-15ed-47a7-8dcb-ab27dc5b29c2"
-          (reference "C3") (unit 1)
+          (reference "C?") (unit 1)
         )
         (path "/8d0803ab-15ed-47a7-8dcb-ab27dc5b29c2/225eaee9-8f74-4a38-a94f-717f461ecd54"
@@
   (symbol (lib_id "power:GND") (at 114.3 60.96 0) (unit 1)
     (in_bom yes) (on_board yes) (dnp no) (fields_autoplaced)
-    (property "Reference" "#PWR026" (at 114.3 67.31 0)
+    (property "Reference" "#PWR?" (at 114.3 67.31 0)
       (effects (font (size 1.27 1.27)) hide)
     )
@@
       (project "MVS"
         (path "/8d0803ab-15ed-47a7-8dcb-ab27dc5b29c2"
-          (reference "#PWR026") (unit 1)
+          (reference "#PWR?") (unit 1)
         )
         (path "/8d0803ab-15ed-47a7-8dcb-ab27dc5b29c2/225eaee9-8f74-4a38-a94f-717f461ecd54"
