File: schematics/MV1F-MB-PowerAmp-Neo-FO-Dip.kicad_sch (KiCad schematic)
At the start: 63 parts, among them J1 SPEAKERS, SW2 SW_DIP_x08, U10 NEO-F0, U9 HA13001

Commit message: Typo... and orphan labels remove
Parts:
- renumbered JP1 to JP?
Changed lines of the file:
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@@
   (symbol (lib_id "Jumper:SolderJumper_2_Open") (at 306.07 148.59 0) (unit 1)
     (in_bom yes) (on_board yes) (dnp no)
-    (property "Reference" "JP1" (at 306.07 151.13 0)
+    (property "Reference" "JP?" (at 306.07 151.13 0)
       (effects (font (size 1.27 1.27)))
     )
@@
       (project "MVS"
         (path "/8d0803ab-15ed-47a7-8dcb-ab27dc5b29c2"
-          (reference "JP1") (unit 1)
+          (reference "JP?") (unit 1)
         )
         (path "/8d0803ab-15ed-47a7-8dcb-ab27dc5b29c2/0b42d888-4b79-4625-b2d5-9f4b583469ed"
@@
   (symbol (lib_id "Jumper:SolderJumper_2_Open") (at 35.56 176.53 0) (unit 1)
     (in_bom yes) (on_board yes) (dnp no)
-    (property "Reference" "JP1" (at 35.56 173.99 0)
+    (property "Reference" "JP?" (at 35.56 173.99 0)
       (effects (font (size 1.27 1.27)))
     )
@@
       (project "MVS"
         (path "/8d0803ab-15ed-47a7-8dcb-ab27dc5b29c2"
-          (reference "JP1") (unit 1)
+          (reference "JP?") (unit 1)
         )
         (path "/8d0803ab-15ed-47a7-8dcb-ab27dc5b29c2/0b42d888-4b79-4625-b2d5-9f4b583469ed"
@@
   (symbol (lib_id "Jumper:SolderJumper_2_Open") (at 306.07 153.67 0) (unit 1)
     (in_bom yes) (on_board yes) (dnp no)
-    (property "Reference" "JP1" (at 306.07 156.21 0)
+    (property "Reference" "JP?" (at 306.07 156.21 0)
       (effects (font (size 1.27 1.27)))
     )
@@
       (project "MVS"
         (path "/8d0803ab-15ed-47a7-8dcb-ab27dc5b29c2"
-          (reference "JP1") (unit 1)
+          (reference "JP?") (unit 1)
         )
         (path "/8d0803ab-15ed-47a7-8dcb-ab27dc5b29c2/0b42d888-4b79-4625-b2d5-9f4b583469ed"
